Commit message: Add panda_ftsensor_robotiq description package
대상 로봇(Panda + FT 센서 + Robotiq 2F-85)의 URDF·메시를 전용 description
패키지로 정리했다. 코드가 없는 자산 전용 패키지이므로 계층 경계와 무관하다.

패키지 이름을 벤더 URDF 의 `package://` 참조와 같게 맞춘 것이 핵심이다.
다르게 두면 메시 경로를 매번 손으로 고쳐야 하는데, 이미 개정본을 한 번 받은
만큼(아래) 그 수정이 누락될 여지를 남기지 않는다.

URDF 개정본 반영 — 관절 한계 3건 정정
- left_inner_finger / right_inner_knuckle / right_outer_knuckle 의 한계가
  [0, 0.8757] → [-0.8757, 0] 로 바뀌었다. 정정된 셋이 정확히 mimic 배수가
  -1 인 셋이며, 구버전은 정상 동작 전 구간이 한계 밖이었다.
- 이 부호가 시뮬레이터 실측(idx 2·3·4 가 음수)과 일치한다. 덕분에 그리퍼
  인덱스↔관절 매핑이 확정됐다 — 벤더 요청 B-6 의 "남은 확인 사항" 해소.
- 메시 참조가 두 패키지(Panda, robotiq_arg85_description)에서 단일
  panda_ftsensor_robotiq 로 통합되고 확장자가 소문자로 바뀌었다.

메시 — Robotiq 10종
- fine 5종은 새로 확보한 것이다. coarse 4종은 기존 저장소 파일과 md5 동일.
- inner_finger_coarse 는 벤더가 .obj 로 주었으나 URDF 는 .stl 을 참조한다.
  기존 STL 이 삼각형 236개·bbox 소수점 6자리까지 일치해 그것을 썼고, 벤더
  원본 .obj 도 함께 보존했다.

제거 — 신규 패키지로 대체됨
- config/panda_ftsensor_robotiq.urdf (관절 한계가 틀린 구버전)
- config/robotiq_arg85_description/ (coarse 5종이 신규에 동일하게 포함됨을
  md5 로 확인한 뒤 제거. Unity .meta 파일은 ROS 쪽에서 쓰지 않는다)

남은 것 — 벤더 요청 B-8 신설
Panda 링크 메시 link0~7.obj 8종이 없어 URDF 로드가 완결되지 않는다.
moveit_resources_panda_description 에 같은 부품이 STL 로 있으나 시뮬레이터가
쓰는 기하와 같다는 보장이 없다 — 다르면 MoveIt 충돌 검사가 실물과 어긋나는데
계획은 성공하고 실행에서만 부딪히므로 에러 없이 드러나지 않는다. 임의 대체
대신 벤더에 요청한다.

Co-Authored-By: Claude Opus 5 <noreply@anthropic.com>

File: src/panda_ftsensor_robotiq/urdf/panda_ftsensor_robotiq.urdf (robot description, URDF)
Before this commit: robot panda, 17 links, 16 joints
Links:
- link left_inner_finger: geometry collision mesh filename=package://panda_ftsensor_robotiq/meshes/inner_finger_coarse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; visual mesh filename=package://panda_ftsensor_robotiq/meshes/inner_finger_fine.s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
- link left_inner_knuckle: geometry collision mesh filename=package://panda_ftsensor_robotiq/meshes/inner_knuckle_coars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; visual mesh filename=package://panda_ftsensor_robotiq/meshes/inner_knuckle_fine.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
- link left_outer_finger: geometry collision mesh filename=package://panda_ftsensor_robotiq/meshes/outer_finger_coarse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; visual mesh filename=package://panda_ftsensor_robotiq/meshes/outer_finger_fine.s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
- link left_outer_knuckle: geometry collision mesh filename=package://panda_ftsensor_robotiq/meshes/outer_knuckle_coars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; visual mesh filename=package://panda_ftsensor_robotiq/meshes/outer_knuckle_fine.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
- link panda_link0: geometry collision mesh filename=package://panda_ftsensor_robotiq/meshes/collision/link0.obj; visual mesh filename=package://panda_ftsensor_robotiq/meshes/collision/link0.obj
- link panda_link1: geometry collision mesh filename=package://panda_ftsensor_robotiq/meshes/collision/link1.obj; visual mesh filename=package://panda_ftsensor_robotiq/meshes/collision/link1.obj
- link panda_link2: geometry collision mesh filename=package://panda_ftsensor_robotiq/meshes/collision/link2.obj; visual mesh filename=package://panda_ftsensor_robotiq/meshes/collision/link2.obj
- link panda_link3: geometry collision mesh filename=package://panda_ftsensor_robotiq/meshes/collision/link3.obj; visual mesh filename=package://panda_ftsensor_robotiq/meshes/collision/link3.obj
- link panda_link4: geometry collision mesh filename=package://panda_ftsensor_robotiq/meshes/collision/link4.obj; visual mesh filename=package://panda_ftsensor_robotiq/meshes/collision/link4.obj
- link panda_link5: geometry collision mesh filename=package://panda_ftsensor_robotiq/meshes/collision/link5.obj; visual mesh filename=package://panda_ftsensor_robotiq/meshes/collision/link5.obj
- link panda_link6: geometry collision mesh filename=package://panda_ftsensor_robotiq/meshes/collision/link6.obj; visual mesh filename=package://panda_ftsensor_robotiq/meshes/collision/link6.obj
- link panda_link7: geometry collision mesh filename=package://panda_ftsensor_robotiq/meshes/collision/link7.obj; visual mesh filename=package://panda_ftsensor_robotiq/meshes/collision/link7.obj
- link right_inner_finger: geometry collision mesh filename=package://panda_ftsensor_robotiq/meshes/inner_finger_coarse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; visual mesh filename=package://panda_ftsensor_robotiq/meshes/inner_finger_fine.s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
- link right_inner_knuckle: geometry collision mesh filename=package://panda_ftsensor_robotiq/meshes/inner_knuckle_coars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; visual mesh filename=package://panda_ftsensor_robotiq/meshes/inner_knuckle_fine.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
- link right_outer_finger: geometry collision mesh filename=package://panda_ftsensor_robotiq/meshes/outer_finger_coarse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; visual mesh filename=package://panda_ftsensor_robotiq/meshes/outer_finger_fine.s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
- link right_outer_knuckle: geometry collision mesh filename=package://panda_ftsensor_robotiq/meshes/outer_knuckle_coars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; visual mesh filename=package://panda_ftsensor_robotiq/meshes/outer_knuckle_fine.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
- link robotiq_85_base_link: geometry collision mesh filename=package://panda_ftsensor_robotiq/meshes/robotiq_85_base_lin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; visual mesh filename=package://panda_ftsensor_robotiq/meshes/robotiq_85_base_lin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
Joints:
- joint left_inner_finger_joint: limit lower=0 upper=0.8757 effort=1000 velocity=2.0 -> lower=-0.8757 upper=0 effort=1000 velocity=2.0
- joint right_inner_knuckle_joint: limit lower=0 upper=0.8757 effort=1000 velocity=2.0 -> lower=-0.8757 upper=0 effort=1000 velocity=2.0
- joint right_outer_knuckle_joint: limit lower=0 upper=0.8757 effort=1000 velocity=2.0 -> lower=-0.8757 upper=0 effort=1000 velocity=2.0
