Commit message: Introduce backend profiles, and the fixes measured on top of them
This is a large accumulated change set — several days of interleaved work that
was never committed. The pieces share files (panda_functionbay.launch.py alone
carries profile, gravity and camera changes), so splitting it by topic would
produce commits that do not build. Code, config and scripts go together here;
docs follow separately.

Backend profiles
  config/backends/<name>.yaml now holds everything that differs per backend —
  arm command channel, ros2_control wiring, simulator topics, servo, camera,
  scene, frames. get_backend('isaac') is the single entry point; `factory:`
  selects a subclass only where a value cannot map to one parameter. Launches
  keep their LaunchConfiguration wiring and take defaults from the profile, so
  overrides like servo_linear_scale:=0.8 still work. Verified by exec'ing each
  launch and diffing argument defaults and servo parameters before/after.

  Consumers stop guessing: create_move_group_client(node, backend=...) and the
  twin's moveit.backend read the same table. Runtime JTC/JGPC detection
  mis-read FunctionBay as JTC, where planning succeeded and execution silently
  did nothing.

Isaac — the servo ratchet
  Servo re-based on the measured state in two places: moveit_servo itself, and
  JTC restarting interpolation from the measured state on every single-point
  trajectory. Load-induced droop was integrated into the command, so holding a
  100 g block and commanding +z drifted 30 mm sideways. commanded_joint_state_node
  feeds servo the controller's commanded position, and a local controllers yaml
  sets open_loop_control: true. Sideways/vertical ratio 0.83 -> 0.01. Servo got
  2.7x faster as a side effect, so teleop's linear/angular step defaults drop to
  0.25.

FunctionBay
  - gravity compensation computed from the vendor URDF and the scene's Kp,
    applied to every streamed command point (12.37 -> 0.00 mm over 8 points).
    This replaces the per-point sag calibration, which is deleted.
  - gripper command profile per scene: axis count, units and packing all differ
    between Crisp and RecurDyn builds. Sending radians to a degree scene moved
    1.7% and looked like a vendor defect.
  - fixtures (holes, trays) live in a config file because the vendor exports TF
    only for non-static bodies; the twin exposes them as a state variable.
  - compressed camera: the new build publishes CompressedImage, so the viewer
    gets a republish companion and the recorder gained an mjpeg input path.

Also: JGPC streaming takes publish_rate from the profile (10 Hz stepping broke
0.5 mm peg insertion), teleop key-hold detection split into key_hold.py, and a
set of measurement scripts under scripts/functionbay and scripts/isaac.

Build and the three suites pass: 1384 tests, 9 skipped.

Co-Authored-By: Claude Opus 5 <noreply@anthropic.com>

File: src/robot_control/description/panda.ros2_control.xacro (robot description, xacro)
@@ -3,8 +3,12 @@
   moveit_resources_panda_moveit_config 의 panda.ros2_control.xacro 를 포크하여
   `gazebo` (ign_ros2_control) 하드웨어 분기를 추가한 버전이다. mock_components /
-  isaac 분기는 원본과 동일하게 유지한다.
+  isaac 분기는 원본과 동일하게 유지한다 (팔에는 effort 를 두지 않는다 —
+  파지 판정에 필요한 것은 손가락뿐이다. panda_hand.ros2_control.xacro 를 본다).
 -->
 <robot xmlns:xacro="http://www.ros.org/wiki/xacro">
-    <xacro:macro name="panda_ros2_control" params="name initial_positions_file ros2_control_hardware_type">
+    <xacro:macro name="panda_ros2_control"
+                 params="name initial_positions_file ros2_control_hardware_type
+                         isaac_joint_commands_topic:=/isaac_joint_commands
+                         isaac_joint_states_topic:=/isaac_joint_states">
         <xacro:property name="initial_positions" value="${xacro.load_yaml(initial_positions_file)['initial_positions']}"/>
         <ros2_control name="${name}" type="system">
@@ -15,6 +19,10 @@
                 <xacro:if value="${ros2_control_hardware_type == 'isaac'}">
                     <plugin>topic_based_ros2_control/TopicBasedSystem</plugin>
-                    <param name="joint_commands_topic">/isaac_joint_commands</param>
-                    <param name="joint_states_topic">/isaac_joint_states</param>
+                    <!-- 토픽 이름은 상위에서 주입한다. Isaac 그래프가 팔·손을 **다른
+                         토픽**으로 받으므로(각각 ArticulationController 가 붙어 있다)
+                         두 시스템이 같은 이름을 쓰면 한쪽이 굶는다. 기본값은 상위
+                         MoveIt 원본과 같다. -->
+                    <param name="joint_commands_topic">${isaac_joint_commands_topic}</param>
+                    <param name="joint_states_topic">${isaac_joint_states_topic}</param>
                 </xacro:if>
                 <xacro:if value="${ros2_control_hardware_type == 'gazebo'}">

File: src/robot_control/description/panda.urdf.xacro (robot description, xacro)
@@ -1,16 +1,22 @@
 <?xml version="1.0"?>
 <!--
-  rdfp 패키지용 Panda 최상위 URDF xacro.
+  robot_control 패키지용 Panda 최상위 URDF xacro. **모든 백엔드의 단일 출처다**
+  (`launch_helpers.common.build_moveit_config()` 가 이것을 읽는다).
   moveit_resources 의 원본 구조를 따르되, 다음을 추가한다.
   - 물리 시뮬레이션용 inertial 이 보강된 링크(panda_links.urdf.xacro).
   - ros2_control 하드웨어 분기에 `gazebo`(ign_ros2_control) 추가.
   - `gazebo` 선택 시 ign_ros2_control 시스템 플러그인 + (옵션) 카메라 센서.
-  mock_components / isaac 로 빌드하면 기존 mock 스택과 동일한 robot_description
-  을 생성한다(추가된 inertial 은 mock 동작에 무해). 즉 단일 description 으로
-  mock / gazebo / isaac 백엔드를 모두 커버한다.
+  moveit_resources 원본과 링크·관절·한계·충돌형상이 완전히 같다(구조 비교로
+  확인). 더해지는 것은 inertial 12개와 하드웨어 분기뿐이며, inertial 은
+  mock 동작에 무해하다.
 -->
 <robot xmlns:xacro="http://www.ros.org/wiki/xacro" name="panda">
-    <xacro:arg name="initial_positions_file" default="$(find rdfp)/description/initial_positions.yaml" />
+    <xacro:arg name="initial_positions_file" default="$(find robot_control)/description/initial_positions.yaml" />
     <xacro:arg name="ros2_control_hardware_type" default="mock_components" />
+    <!-- isaac(plugin) 백엔드에서 TopicBasedSystem 이 쓸 토픽. 팔과 손이 다른 것은
+         Isaac 그래프가 둘을 따로 받기 때문이다. bridge 방식에서는 쓰이지 않는다. -->
+    <xacro:arg name="isaac_arm_command_topic" default="/isaac_joint_commands" />
+    <xacro:arg name="isaac_gripper_command_topic" default="/isaac_joint_commands" />
+    <xacro:arg name="isaac_joint_states_topic" default="/isaac_joint_states" />
     <!-- gazebo 백엔드에서 ign_ros2_control 플러그인에 넘길 컨트롤러 YAML 절대경로. -->
     <xacro:arg name="ros2_controllers_file" default="$(find moveit_resources_panda_moveit_config)/config/ros2_controllers.yaml" />
@@ -18,13 +24,19 @@
     <xacro:arg name="simulate_camera" default="false" />
     <!-- 링크/조인트 + inertial (geometry 는 moveit_resources 메시 참조) -->
-    <xacro:include filename="$(find rdfp)/description/panda_links.urdf.xacro" />
+    <xacro:include filename="$(find robot_control)/description/panda_links.urdf.xacro" />
     <!-- ros2_control description -->
-    <xacro:include filename="$(find rdfp)/description/panda.ros2_control.xacro" />
-    <xacro:include filename="$(find rdfp)/description/panda_hand.ros2_control.xacro" />
-    <xacro:panda_ros2_control name="PandaSystem" initial_positions_file="$(arg initial_positions_file)" ros2_control_hardware_type="$(arg ros2_control_hardware_type)" />
-    <xacro:panda_hand_ros2_control name="PandaHandSystem" ros2_control_hardware_type="$(arg ros2_control_hardware_type)" />
+    <xacro:include filename="$(find robot_control)/description/panda.ros2_control.xacro" />
+    <xacro:include filename="$(find robot_control)/description/panda_hand.ros2_control.xacro" />
+    <xacro:panda_ros2_control name="PandaSystem" initial_positions_file="$(arg initial_positions_file)"
+                              ros2_control_hardware_type="$(arg ros2_control_hardware_type)"
+                              isaac_joint_commands_topic="$(arg isaac_arm_command_topic)"
+                              isaac_joint_states_topic="$(arg isaac_joint_states_topic)" />
+    <xacro:panda_hand_ros2_control name="PandaHandSystem"
+                                   ros2_control_hardware_type="$(arg ros2_control_hardware_type)"
+                                   isaac_joint_commands_topic="$(arg isaac_gripper_command_topic)"
+                                   isaac_joint_states_topic="$(arg isaac_joint_states_topic)" />
     <!-- gazebo 전용: ign_ros2_control 시스템 플러그인 + (옵션) 카메라 -->
     <xacro:if value="${'$(arg ros2_control_hardware_type)' == 'gazebo'}">
-        <xacro:include filename="$(find rdfp)/description/panda.gazebo.xacro" />
+        <xacro:include filename="$(find robot_control)/description/panda.gazebo.xacro" />
         <xacro:panda_world_anchor />
         <xacro:panda_gazebo_ros2_control ros2_controllers_file="$(arg ros2_controllers_file)" />

File: src/robot_control/description/panda_hand.ros2_control.xacro (robot description, xacro)
@@ -2,8 +2,12 @@
 <!--
   moveit_resources_panda_moveit_config 의 panda_hand.ros2_control.xacro 를
-  포크하여 `gazebo` (ign_ros2_control) 하드웨어 분기를 추가한 버전이다.
+  포크하여 `gazebo` (ign_ros2_control) 하드웨어 분기와, `isaac` 한정
+  effort state_interface 를 추가한 버전이다.
 -->
 <robot xmlns:xacro="http://www.ros.org/wiki/xacro">
-    <xacro:macro name="panda_hand_ros2_control" params="name ros2_control_hardware_type">
+    <xacro:macro name="panda_hand_ros2_control"
+                 params="name ros2_control_hardware_type
+                         isaac_joint_commands_topic:=/isaac_joint_commands
+                         isaac_joint_states_topic:=/isaac_joint_states">
         <ros2_control name="${name}" type="system">
             <hardware>
@@ -13,6 +17,10 @@
                 <xacro:if value="${ros2_control_hardware_type == 'isaac'}">
                     <plugin>topic_based_ros2_control/TopicBasedSystem</plugin>
-                    <param name="joint_commands_topic">/isaac_joint_commands</param>
-                    <param name="joint_states_topic">/isaac_joint_states</param>
+                    <!-- 토픽 이름은 상위에서 주입한다. Isaac 그래프가 팔·손을 **다른
+                         토픽**으로 받으므로(각각 ArticulationController 가 붙어 있다)
+                         두 시스템이 같은 이름을 쓰면 한쪽이 굶는다. 기본값은 상위
+                         MoveIt 원본과 같다. -->
+                    <param name="joint_commands_topic">${isaac_joint_commands_topic}</param>
+                    <param name="joint_states_topic">${isaac_joint_states_topic}</param>
                 </xacro:if>
                 <xacro:if value="${ros2_control_hardware_type == 'gazebo'}">
@@ -28,4 +36,14 @@
                     <param name="initial_value">0.0</param>
                 </state_interface>
+                <!-- effort 는 isaac 에서만 싣는다. `grasp` 의 at_goal 판정이
+                     GripperNode 의 stall_effort 로 이뤄지는데, 그 값의 출처가
+                     이 인터페이스다. mock 은 손가락 effort 를 만들어내지 못해
+                     (GenericSystem 이 0 을 보고한다) 켜면 '항상 안 물림'이라는
+                     거짓을 말하므로 넣지 않는다. -->
+                <xacro:if value="${ros2_control_hardware_type == 'isaac'}">
+                    <state_interface name="effort">
+                        <param name="initial_value">0.0</param>
+                    </state_interface>
+                </xacro:if>
             </joint>
             <!-- panda_finger_joint2 는 finger_joint1 을 mimic 한다. ign_ros2_control
@@ -43,4 +61,9 @@
                     <param name="initial_value">0.0</param>
                 </state_interface>
+                <xacro:if value="${ros2_control_hardware_type == 'isaac'}">
+                    <state_interface name="effort">
+                        <param name="initial_value">0.0</param>
+                    </state_interface>
+                </xacro:if>
             </joint>
         </ros2_control>
